Commit message: DH Grippers added

File: urdf/overseas_65_b_v_description.urdf (robot description, URDF)
Before this commit: robot overseas_65_b_v_description, 33 links, 32 joints
Links:
- removed link l_hand_base_link
- removed link r_hand_base_link
- added link l_gripper_base_link, mass 0.83416; collision mesh filename=visual/base_link.STL scale=0.001 0.001 0.001; visual mesh filename=visual/base_link.STL scale=0.001 0.001 0.001
- added link l_gripper_finger1_finger_link, mass 0.0222871; collision mesh filename=visual/rod_Link.STL scale=0.001 0.001 0.001; visual mesh filename=visual/rod_Link.STL scale=0.001 0.001 0.001
- added link l_gripper_finger1_finger_tip_link, mass 0.0124305; collision mesh filename=visual/distal_phalanx_Link.STL scale=0.001 0.001 0.001; visual mesh filename=visual/distal_phalanx_Link.STL scale=0.001 0.001 0.001
- added link l_gripper_finger1_inner_knuckle_link, mass 0.0318004; collision mesh filename=visual/proximal_phalanx_Link.STL scale=0.001 0.001 0.001; visual mesh filename=visual/proximal_phalanx_Link.STL scale=0.001 0.001 0.001
- added link l_gripper_finger1_knuckle_link, mass 0.011111; collision mesh filename=visual/crank_Link.STL scale=0.001 0.001 0.001; visual mesh filename=visual/crank_Link.STL scale=0.001 0.001 0.001
- added link l_gripper_finger2_finger_link, mass 0.0222871; collision mesh filename=visual/rod_Link.STL scale=0.001 0.001 0.001; visual mesh filename=visual/rod_Link.STL scale=0.001 0.001 0.001
- added link l_gripper_finger2_finger_tip_link, mass 0.0124305; collision mesh filename=visual/distal_phalanx_Link.STL scale=0.001 0.001 0.001; visual mesh filename=visual/distal_phalanx_Link.STL scale=0.001 0.001 0.001
- added link l_gripper_finger2_inner_knuckle_link, mass 0.0318004; collision mesh filename=visual/proximal_phalanx_Link.STL scale=0.001 0.001 0.001; visual mesh filename=visual/proximal_phalanx_Link.STL scale=0.001 0.001 0.001
- added link l_gripper_finger2_knuckle_link, mass 0.011111; collision mesh filename=visual/crank_Link.STL scale=0.001 0.001 0.001; visual mesh filename=visual/crank_Link.STL scale=0.001 0.001 0.001
- added link r_gripper_base_link, mass 0.83416; collision mesh filename=visual/base_link.STL scale=0.001 0.001 0.001; visual mesh filename=visual/base_link.STL scale=0.001 0.001 0.001
- added link r_gripper_finger1_finger_link, mass 0.0222871; collision mesh filename=visual/rod_Link.STL scale=0.001 0.001 0.001; visual mesh filename=visual/rod_Link.STL scale=0.001 0.001 0.001
- added link r_gripper_finger1_finger_tip_link, mass 0.0124305; collision mesh filename=visual/distal_phalanx_Link.STL scale=0.001 0.001 0.001; visual mesh filename=visual/distal_phalanx_Link.STL scale=0.001 0.001 0.001
- added link r_gripper_finger1_inner_knuckle_link, mass 0.0318004; collision mesh filename=visual/proximal_phalanx_Link.STL scale=0.001 0.001 0.001; visual mesh filename=visual/proximal_phalanx_Link.STL scale=0.001 0.001 0.001
- added link r_gripper_finger1_knuckle_link, mass 0.011111; collision mesh filename=visual/crank_Link.STL scale=0.001 0.001 0.001; visual mesh filename=visual/crank_Link.STL scale=0.001 0.001 0.001
- added link r_gripper_finger2_finger_link, mass 0.0222871; collision mesh filename=visual/rod_Link.STL scale=0.001 0.001 0.001; visual mesh filename=visual/rod_Link.STL scale=0.001 0.001 0.001
- added link r_gripper_finger2_finger_tip_link, mass 0.0124305; collision mesh filename=visual/distal_phalanx_Link.STL scale=0.001 0.001 0.001; visual mesh filename=visual/distal_phalanx_Link.STL scale=0.001 0.001 0.001
- added link r_gripper_finger2_inner_knuckle_link, mass 0.0318004; collision mesh filename=visual/proximal_phalanx_Link.STL scale=0.001 0.001 0.001; visual mesh filename=visual/proximal_phalanx_Link.STL scale=0.001 0.001 0.001
- added link r_gripper_finger2_knuckle_link, mass 0.011111; collision mesh filename=visual/crank_Link.STL scale=0.001 0.001 0.001; visual mesh filename=visual/crank_Link.STL scale=0.001 0.001 0.001
- link base_link_underpan: geometry collision mesh filename=meshes/base_link_underpan.STL; visual mesh filename=meshes/base_link_underpan.STL
- link body_base_link: geometry collision mesh filename=meshes/body_base_link.STL; visual mesh filename=meshes/body_base_link.STL
- link camera_link: geometry collision mesh filename=meshes/camera_link.STL; visual mesh filename=meshes/camera_link.STL
- link head_link1: geometry collision mesh filename=meshes/head_link1.STL; visual mesh filename=meshes/head_link1.STL
- link head_link2: geometry collision mesh filename=meshes/head_link2.STL; visual mesh filename=meshes/head_link2.STL
- link l_base_link1: geometry collision mesh filename=meshes/l_base_link1.STL; visual mesh filename=meshes/l_base_link1.STL
- link l_link1: geometry collision mesh filename=meshes/l_link1.STL; visual mesh filename=meshes/l_link1.STL
- link l_link2: geometry collision mesh filename=meshes/l_link2.STL; visual mesh filename=meshes/l_link2.STL
- link l_link3: geometry collision mesh filename=meshes/l_link3.STL; visual mesh filename=meshes/l_link3.STL
- link l_link4: geometry collision mesh filename=meshes/l_link4.STL; visual mesh filename=meshes/l_link4.STL
- link l_link5: geometry collision mesh filename=meshes/l_link5.STL; visual mesh filename=meshes/l_link5.STL
- link l_link6: geometry collision mesh filename=meshes/l_link6.STL; visual mesh filename=meshes/l_link6.STL
- link link_left_wheel: geometry collision mesh filename=meshes/link_left_wheel.STL; visual mesh filename=meshes/link_left_wheel.STL
- link link_right_wheel: geometry collision mesh filename=meshes/link_right_wheel.STL; visual mesh filename=meshes/link_right_wheel.STL
- link link_swivel_wheel_1_1: geometry collision mesh filename=meshes/link_swivel_wheel_1_1.STL; visual mesh filename=meshes/link_swivel_wheel_1_1.STL
- link link_swivel_wheel_1_2: geometry collision mesh filename=meshes/link_swivel_wheel_1_2.STL; visual mesh filename=meshes/link_swivel_wheel_1_2.STL
- link link_swivel_wheel_2_1: geometry collision mesh filename=meshes/link_swivel_wheel_2_1.STL; visual mesh filename=meshes/link_swivel_wheel_2_1.STL
- link link_swivel_wheel_2_2: geometry collision mesh filename=meshes/link_swivel_wheel_2_2.STL; visual mesh filename=meshes/link_swivel_wheel_2_2.STL
- link link_swivel_wheel_3_1: geometry collision mesh filename=meshes/link_swivel_wheel_3_1.STL; visual mesh filename=meshes/link_swivel_wheel_3_1.STL
- link link_swivel_wheel_3_2: geometry collision mesh filename=meshes/link_swivel_wheel_3_2.STL; visual mesh filename=meshes/link_swivel_wheel_3_2.STL
- link link_swivel_wheel_4_1: geometry collision mesh filename=meshes/link_swivel_wheel_4_1.STL; visual mesh filename=meshes/link_swivel_wheel_4_1.STL
- link link_swivel_wheel_4_2: geometry collision mesh filename=meshes/link_swivel_wheel_4_2.STL; visual mesh filename=meshes/link_swivel_wheel_4_2.STL
- link platform_base_link: geometry collision mesh filename=meshes/platform_base_link.STL; visual mesh filename=meshes/platform_base_link.STL
- link r_base_link1: geometry collision mesh filename=meshes/r_base_link1.STL; visual mesh filename=meshes/r_base_link1.STL
- link r_link1: geometry collision mesh filename=meshes/r_link1.STL; visual mesh filename=meshes/r_link1.STL
- link r_link2: geometry collision mesh filename=meshes/r_link2.STL; visual mesh filename=meshes/r_link2.STL
- link r_link3: geometry collision mesh filename=meshes/r_link3.STL; visual mesh filename=meshes/r_link3.STL
- link r_link4: geometry collision mesh filename=meshes/r_link4.STL; visual mesh filename=meshes/r_link4.STL
- link r_link5: geometry collision mesh filename=meshes/r_link5.STL; visual mesh filename=meshes/r_link5.STL
- link r_link6: geometry collision mesh filename=meshes/r_link6.STL; visual mesh filename=meshes/r_link6.STL
Joints:
- added joint l_gripper_finger1_finger_joint: type continuous, parent l_gripper_finger1_knuckle_link, child l_gripper_finger1_finger_link, origin xyz=0.0292080077784 0.0 -0.0227132622407 rpy=0 0 0, axis 0 -1 0, limit lower=-3.14 upper=3.14 effort=0.1 velocity=100.0, mimic joint=l_gripper_finger1_joint multiplier=0.4563942 offset=0
- added joint l_gripper_finger1_finger_tip_joint: type continuous, parent l_gripper_finger1_inner_knuckle_link, child l_gripper_finger1_finger_tip_link, origin xyz=0.0394969463769 0.0 0.0382752038125  rpy=0.0 0.0 0.0, axis 0 1 0, limit lower=-3.14 upper=3.14 effort=0.1 velocity=100.0, mimic joint=l_gripper_finger1_joint multiplier=1.49462955
- added joint l_gripper_finger1_inner_knuckle_joint: type continuous, parent l_gripper_base_link, child l_gripper_finger1_inner_knuckle_link, origin xyz=-0.016 0 0.10586 rpy=0.0 0.0 3.14, axis 0 -1 0, limit lower=-3.14 upper=3.14 effort=0.1 velocity=100.0, mimic joint=l_gripper_finger1_joint multiplier=1.49462955 offset=0
- added joint l_gripper_finger1_joint: type revolute, parent l_gripper_base_link, child l_gripper_finger1_knuckle_link, origin xyz=-0.016 0 0.10586 rpy=0.0 0.0 3.14, axis 0 -1 0, limit lower=0.0 upper=0.6524 effort=1000 velocity=2.0
- added joint l_gripper_finger2_finger_joint: type continuous, parent l_gripper_finger2_knuckle_link, child l_gripper_finger2_finger_link, origin xyz=0.0292080077784 0.0 -0.0227132622407 rpy=0 0 0, axis 0 -1 0, limit lower=-3.14 upper=3.14 effort=0.1 velocity=100.0, mimic joint=l_gripper_finger1_joint multiplier=0.4563942 offset=0
- added joint l_gripper_finger2_finger_tip_joint: type continuous, parent l_gripper_finger2_inner_knuckle_link, child l_gripper_finger2_finger_tip_link, origin xyz=0.0394969463769  0.0 0.0382752038125   rpy=0.0 0.0 0.0, axis 0 1 0, limit lower=-3.14 upper=3.14 effort=0.1 velocity=100.0, mimic joint=l_gripper_finger1_joint multiplier=1.49462955
- added joint l_gripper_finger2_inner_knuckle_joint: type continuous, parent l_gripper_base_link, child l_gripper_finger2_inner_knuckle_link, origin xyz=0.016 0 0.10586 rpy=0.0 0.0 0.0, axis 0 -1 0, limit lower=-3.14 upper=3.14 effort=0.1 velocity=100.0, mimic joint=l_gripper_finger1_joint multiplier=1.49462955 offset=0
- added joint l_gripper_finger2_joint: type revolute, parent l_gripper_base_link, child l_gripper_finger2_knuckle_link, origin xyz=0.016  0 0.10586  rpy=0.0 0.0 0.0, axis 0 -1 0, limit lower=-3.14 upper=3.14 effort=1000 velocity=100.0, mimic joint=l_gripper_finger1_joint
- added joint r_gripper_finger1_finger_joint: type continuous, parent r_gripper_finger1_knuckle_link, child r_gripper_finger1_finger_link, origin xyz=0.0292080077784 0.0 -0.0227132622407 rpy=0 0 0, axis 0 -1 0, limit lower=-3.14 upper=3.14 effort=0.1 velocity=100.0, mimic joint=r_gripper_finger1_joint multiplier=0.4563942 offset=0
- added joint r_gripper_finger1_finger_tip_joint: type continuous, parent r_gripper_finger1_inner_knuckle_link, child r_gripper_finger1_finger_tip_link, origin xyz=0.0394969463769 0.0 0.0382752038125  rpy=0.0 0.0 0.0, axis 0 1 0, limit lower=-3.14 upper=3.14 effort=0.1 velocity=100.0, mimic joint=r_gripper_finger1_joint multiplier=1.49462955
- added joint r_gripper_finger1_inner_knuckle_joint: type continuous, parent r_gripper_base_link, child r_gripper_finger1_inner_knuckle_link, origin xyz=-0.016 0 0.10586 rpy=0.0 0.0 3.14, axis 0 -1 0, limit lower=-3.14 upper=3.14 effort=0.1 velocity=100.0, mimic joint=r_gripper_finger1_joint multiplier=1.49462955 offset=0
- added joint r_gripper_finger1_joint: type revolute, parent r_gripper_base_link, child r_gripper_finger1_knuckle_link, origin xyz=-0.016 0 0.10586 rpy=0.0 0.0 3.14, axis 0 -1 0, limit lower=0.0 upper=0.6524 effort=1000 velocity=2.0
- added joint r_gripper_finger2_finger_joint: type continuous, parent r_gripper_finger2_knuckle_link, child r_gripper_finger2_finger_link, origin xyz=0.0292080077784 0.0 -0.0227132622407 rpy=0 0 0, axis 0 -1 0, limit lower=-3.14 upper=3.14 effort=0.1 velocity=100.0, mimic joint=r_gripper_finger1_joint multiplier=0.4563942 offset=0
- added joint r_gripper_finger2_finger_tip_joint: type continuous, parent r_gripper_finger2_inner_knuckle_link, child r_gripper_finger2_finger_tip_link, origin xyz=0.0394969463769  0.0 0.0382752038125   rpy=0.0 0.0 0.0, axis 0 1 0, limit lower=-3.14 upper=3.14 effort=0.1 velocity=100.0, mimic joint=l_gripper_finger1_joint multiplier=1.49462955
- added joint r_gripper_finger2_inner_knuckle_joint: type continuous, parent r_gripper_base_link, child r_gripper_finger2_inner_knuckle_link, origin xyz=0.016 0 0.10586 rpy=0.0 0.0 0.0, axis 0 -1 0, limit lower=-3.14 upper=3.14 effort=0.1 velocity=100.0, mimic joint=r_gripper_finger1_joint multiplier=1.49462955 offset=0
- added joint r_gripper_finger2_joint: type revolute, parent r_gripper_base_link, child r_gripper_finger2_knuckle_link, origin xyz=0.016  0 0.10586  rpy=0.0 0.0 0.0, axis 0 -1 0, limit lower=-3.14 upper=3.14 effort=1000 velocity=100.0, mimic joint=r_gripper_finger1_joint
- joint l_hand_joint: child l_hand_base_link -> l_gripper_base_link; origin xyz=0 0 0.0445 rpy=0 3.1415 3.1415 -> xyz=0 0 0.0445 rpy=3.14159 0 0
- joint r_hand_joint: child r_hand_base_link -> r_gripper_base_link
