Commit message: add pinnocho

File: urdf/overseas_65_corrected.urdf (robot description, URDF)
Before this commit: robot overseas_65_b_v_description, 20 links, 19 joints
Links:
- added link link_left_wheel, mass 1.0734; collision mesh filename=meshes/link_left_wheel.STL; visual mesh filename=meshes/link_left_wheel.STL
- added link link_right_wheel, mass 1.0523; collision mesh filename=meshes/link_right_wheel.STL; visual mesh filename=meshes/link_right_wheel.STL
- added link link_swivel_wheel_1_1, mass 0.088835; collision mesh filename=meshes/link_swivel_wheel_1_1.STL; visual mesh filename=meshes/link_swivel_wheel_1_1.STL
- added link link_swivel_wheel_1_2, mass 0.12664; collision mesh filename=meshes/link_swivel_wheel_1_2.STL; visual mesh filename=meshes/link_swivel_wheel_1_2.STL
- added link link_swivel_wheel_2_1, mass 0.088835; collision mesh filename=meshes/link_swivel_wheel_2_1.STL; visual mesh filename=meshes/link_swivel_wheel_2_1.STL
- added link link_swivel_wheel_2_2, mass 0.12664; collision mesh filename=meshes/link_swivel_wheel_2_2.STL; visual mesh filename=meshes/link_swivel_wheel_2_2.STL
- added link link_swivel_wheel_3_1, mass 0.088835; collision mesh filename=meshes/link_swivel_wheel_3_1.STL; visual mesh filename=meshes/link_swivel_wheel_3_1.STL
- added link link_swivel_wheel_3_2, mass 0.12664; collision mesh filename=meshes/link_swivel_wheel_3_2.STL; visual mesh filename=meshes/link_swivel_wheel_3_2.STL
- added link link_swivel_wheel_4_1, mass 0.088835; collision mesh filename=meshes/link_swivel_wheel_4_1.STL; visual mesh filename=meshes/link_swivel_wheel_4_1.STL
- added link link_swivel_wheel_4_2, mass 0.12664; collision mesh filename=meshes/link_swivel_wheel_4_2.STL; visual mesh filename=meshes/link_swivel_wheel_4_2.STL
Joints:
- added joint joint_left_wheel: type continuous, parent base_link_underpan, child link_left_wheel, origin xyz=0.148 0.015574 -0.153 rpy=0 0 0, axis -1 0 0, limit effort=100 velocity=10
- added joint joint_right_wheel: type continuous, parent base_link_underpan, child link_right_wheel, origin xyz=-0.148 0.015574 -0.153 rpy=0 0 0, axis 1 0 0, limit effort=100 velocity=10
- added joint joint_swivel_wheel_1_1: type continuous, parent base_link_underpan, child link_swivel_wheel_1_1, origin xyz=0.124 -0.17843 -0.16254 rpy=0 0 0, axis 0 0 1
- added joint joint_swivel_wheel_1_2: type continuous, parent link_swivel_wheel_1_1, child link_swivel_wheel_1_2, origin xyz=-0.0035 -0.022 -0.04516 rpy=0 0 0, axis 1 0 0
- added joint joint_swivel_wheel_2_1: type continuous, parent base_link_underpan, child link_swivel_wheel_2_1, origin xyz=-0.126 0.22157 -0.16254 rpy=0 0 0, axis 0 0 1
- added joint joint_swivel_wheel_2_2: type continuous, parent link_swivel_wheel_2_1, child link_swivel_wheel_2_2, origin xyz=-0.0035 -0.022 -0.04516 rpy=0 0 0, axis 1 0 0
- added joint joint_swivel_wheel_3_1: type continuous, parent base_link_underpan, child link_swivel_wheel_3_1, origin xyz=0.124 0.22157 -0.16254 rpy=0 0 0, axis 0 0 1
- added joint joint_swivel_wheel_3_2: type continuous, parent link_swivel_wheel_3_1, child link_swivel_wheel_3_2, origin xyz=-0.0035 -0.022 -0.04516 rpy=0 0 0, axis 1 0 0
- added joint joint_swivel_wheel_4_1: type continuous, parent base_link_underpan, child link_swivel_wheel_4_1, origin xyz=-0.126 -0.17843 -0.1665 rpy=0 0 0, axis 0 0 1
- added joint joint_swivel_wheel_4_2: type continuous, parent link_swivel_wheel_4_1, child link_swivel_wheel_4_2, origin xyz=-0.0035 -0.022 -0.0412 rpy=0 0 0, axis 1 0 0

Commit message: pinochio vis works and sync with isaac, now need to check door mass

File: urdf/overseas_65_corrected.urdf (robot description, URDF)
Before this commit: robot overseas_65_b_v_description, 30 links, 29 joints
Links:
- removed link link_left_wheel
- removed link link_right_wheel
- removed link link_swivel_wheel_1_1
- removed link link_swivel_wheel_1_2
- removed link link_swivel_wheel_2_1
- removed link link_swivel_wheel_2_2
- removed link link_swivel_wheel_3_1
- removed link link_swivel_wheel_3_2
- removed link link_swivel_wheel_4_1
- removed link link_swivel_wheel_4_2
- added link l_gripper_base_link, mass 0.83416; collision mesh filename=visual/base_link.STL scale=0.001 0.001 0.001; visual mesh filename=visual/base_link.STL scale=0.001 0.001 0.001
- added link r_gripper_base_link, mass 0.83416; collision mesh filename=visual/base_link.STL scale=0.001 0.001 0.001; visual mesh filename=visual/base_link.STL scale=0.001 0.001 0.001
Joints:
- removed joint joint_left_wheel
- removed joint joint_right_wheel
- removed joint joint_swivel_wheel_1_1
- removed joint joint_swivel_wheel_1_2
- removed joint joint_swivel_wheel_2_1
- removed joint joint_swivel_wheel_2_2
- removed joint joint_swivel_wheel_3_1
- removed joint joint_swivel_wheel_3_2
- removed joint joint_swivel_wheel_4_1
- removed joint joint_swivel_wheel_4_2
- added joint l_hand_joint: type fixed, parent l_link6, child l_gripper_base_link, origin xyz=0 0 0.0445 rpy=0 0 0, axis 0 0 -1, limit lower=0 upper=0 effort=0 velocity=0
- added joint r_hand_joint: type fixed, parent r_link6, child r_gripper_base_link, origin xyz=0 0 0.0445 rpy=0 0 0, axis 0 0 -1, limit lower=0 upper=0 effort=0 velocity=0

Commit message: pull from ziyi devel

File: urdf/overseas_65_corrected.urdf (robot description, URDF)
Before this commit: robot overseas_65_b_v_description, 22 links, 21 joints
Links:
- added link base_link, mass 0.001
Joints:
- added joint base_rotation_joint: type fixed, parent base_link, child base_link_underpan, origin xyz=0 0 0 rpy=0 0 1.57079

Commit message: removing model initial orientation

File: urdf/overseas_65_corrected.urdf (robot description, URDF)
Before this commit: robot overseas_65_b_v_description, 23 links, 22 joints
Links:
- removed link base_link
Joints:
- removed joint base_rotation_joint

Commit message: added the option to switch to planning in the base local frame

File: urdf/overseas_65_corrected.urdf (robot description, URDF)
Before this commit: robot overseas_65_b_v_description, 22 links, 21 joints
Links:
- link body_base_link: mass 12.159 -> 20
- link platform_base_link: mass 2.8992 -> 5
